Commit message: fixes namespaces

File: gazebo_simulation/urdf/arm_description.urdf (robot description, URDF)
Before this commit: robot myfirst, 5 links, 4 joints
Links:
- link arm_0_bottom: geometry visual mesh filename=package://gazebo_simulation/meshes/arm_0_bottom.stl scale=0.01 0.01 0.01
- link arm_0_top: geometry visual mesh filename=package://gazebo_simulation/meshes/arm_0_top.stl scale=0.01 0.01 0.01
- link arm_1: geometry visual mesh filename=package://gazebo_simulation/meshes/arm_1.stl scale=0.01 0.01 0.01
- link arm_2: geometry visual mesh filename=package://gazebo_simulation/meshes/arm_2.stl scale=0.01 0.01 0.01
- link base_link: geometry visual mesh filename=package://gazebo_simulation/meshes/arm_0_closing_case.stl scale=0.01 0.01 0.01

Commit message: Both arms in rviz

File: gazebo_simulation/urdf/arm_description.urdf (robot description, URDF)
Before this commit: robot arm4DoF, 5 links, 4 joints
Links:
- added link arm_0_closing_case; visual mesh filename=package://gazebo_simulation/meshes/arm_0_closing_case.stl scale=0.01 0.01 0.01
- link base_link: geometry 
Joints:
- added joint arm_0_closing_case_joint: type fixed, parent arm_0_top, child arm_0_closing_case, origin xyz=0 0 -0.07 rpy=0 0 0
- joint arm_0_bottom_joint: parent arm_0_top -> arm_0_closing_case
- joint arm_0_top_joint: limit (none) -> lower=-0.38 upper=0 effort=1000.0 velocity=0.5
