Commit message: Several tries for moveit wrapper. Still not get it working

File: gazebo_simulation/urdf/arm4DoF.urdf (robot description, URDF)
Before this commit: robot arm4DoF, 6 links, 5 joints
Joints:
- joint arm_0_bottom_joint: origin xyz=0 0 -0.335 rpy=0 ${pi/2} 0 -> xyz=0 0 -0.335 rpy=0 1.57079632679 0
- joint arm_1_joint: origin xyz=0 0 0 rpy=${pi/2} 0 ${pi/2} -> xyz=0 0 0 rpy=1.57079632679 0 1.57079632679

Commit message: Not working at all

File: gazebo_simulation/urdf/arm4DoF.urdf (robot description, URDF)
Before this commit: robot arm4DoF, 6 links, 5 joints
Joints:
- joint arm_0_top_joint: limit lower=-0.38 upper=0 effort=1000.0 velocity=0.5 -> (none)
