Commit message: Both arms fixed.

File: arm_description/urdf/arm_description.urdf (robot description, URDF)
Before this commit: robot arm4DoF, 11 links, 10 joints
Links:
- link left/arm_0_bottom: geometry visual mesh filename=package://arm_description/meshes/arm_0_bottom.stl scale=0.01 0.01 0.01
- link left/arm_0_closing_case: geometry visual mesh filename=package://arm_description/meshes/arm_0_closing_case.stl scale=0.01 0.01 0.01
- link left/arm_0_top: geometry collision box size=1 1 0.67; visual mesh filename=package://arm_description/meshes/arm_0_top.stl scale=0.01 0.01 0.01
- link left/arm_1: geometry collision box size=0.73 0.3 1.0; visual mesh filename=package://arm_description/meshes/arm_1.stl scale=0.01 0.01 0.01
- link left/arm_2: geometry collision box size=0.9 0.3 1.3; visual mesh filename=package://arm_description/meshes/arm_2.stl scale=0.01 0.01 0.01
- link right/arm_0_bottom: geometry visual mesh filename=package://arm_description/meshes/arm_0_bottom.stl scale=0.01 0.01 0.01
- link right/arm_0_closing_case: geometry visual mesh filename=package://arm_description/meshes/arm_0_closing_case.stl scale=0.01 0.01 0.01
- link right/arm_0_top: geometry collision box size=1 1 0.67; visual mesh filename=package://arm_description/meshes/arm_0_top.stl scale=0.01 0.01 0.01
- link right/arm_1: geometry collision box size=0.73 0.3 1.0; visual mesh filename=package://arm_description/meshes/arm_1.stl scale=0.01 0.01 0.01
- link right/arm_2: geometry collision box size=0.9 0.3 1.3; visual mesh filename=package://arm_description/meshes/arm_2.stl scale=0.01 0.01 0.01

File: arm_description/urdf/one_arm.urdf (robot description, URDF)
Before this commit: robot arm4DoF, 6 links, 5 joints
Links:
- link arm_0_bottom: geometry visual mesh filename=package://arm_description/meshes/arm_0_bottom.stl scale=0.01 0.01 0.01
- link arm_0_closing_case: geometry visual mesh filename=package://arm_description/meshes/arm_0_closing_case.stl scale=0.01 0.01 0.01
- link arm_0_top: geometry collision box size=1 1 0.67; visual mesh filename=package://arm_description/meshes/arm_0_top.stl scale=0.01 0.01 0.01
- link arm_1: geometry collision box size=0.73 0.3 1.0; visual mesh filename=package://arm_description/meshes/arm_1.stl scale=0.01 0.01 0.01
- link arm_2: geometry collision box size=0.86 0.3 1.2; visual mesh filename=package://arm_description/meshes/arm_2.stl scale=0.01 0.01 0.01
