Commit message: Arm with half of the gripper. Readme file in urdf folder.

File: arm_description/urdf/4dof.urdf (robot description, URDF)
Before this commit: robot arm4DoF, 23 links, 22 joints
Links:
- removed link right/arm_0_attachment
- removed link right/arm_0_bottom
- removed link right/arm_0_bottom_case
- removed link right/arm_0_bottom_top_lock
- removed link right/arm_0_top
- removed link right/arm_1
- removed link right/arm_1_case
- removed link right/arm_2_case_bearing
- removed link right/arm_2_microservo
- removed link right/arm_2_microservo_case
- removed link right/end_effector_connector
- added link left/ScrewActuatorGripper; visual mesh filename=package://arm_description/meshes/new_meshes/gripper/ScrewAc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
- added link left/base_gripper; visual mesh filename=package://arm_description/meshes/new_meshes/gripper/base_gr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
- added link left/core_structure; visual mesh filename=package://arm_description/meshes/new_meshes/gripper/core_st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
- added link left/holdBar_left; visual mesh filename=package://arm_description/meshes/new_meshes/gripper/holdBar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
- added link left/holdBar_right; visual mesh filename=package://arm_description/meshes/new_meshes/gripper/holdBar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
Joints:
- removed joint left/arm_0_bottom_case
- removed joint left/arm_0_bottom_top_lock
- removed joint left/arm_2_case_bearing
- removed joint left/end_effector_connector
- removed joint right/arm_0_attachment_joint
- removed joint right/arm_0_bottom_case
- removed joint right/arm_0_bottom_joint
- removed joint right/arm_0_bottom_top_lock
- removed joint right/arm_0_top_joint
- removed joint right/arm_1_case_joint
- removed joint right/arm_1_joint
- removed joint right/arm_2_case_bearing
- removed joint right/arm_2_microservo_case_joint
- removed joint right/arm_2_microservo_joint
- removed joint right/end_effector_connector
- added joint left/ScrewActuatorGripper_joint: type fixed, parent left/base_gripper, child left/ScrewActuatorGripper, origin xyz=0 0 0.055 rpy=0 0 0
- added joint left/arm_0_bottom_case_joint: type fixed, parent left/arm_0_bottom, child left/arm_0_bottom_case, origin xyz=-0.017 0 0 rpy=0 0 0
- added joint left/arm_0_bottom_top_lock_joint: type fixed, parent left/arm_0_top, child left/arm_0_bottom_top_lock, origin xyz=0 0 0 rpy=0 0 0
- added joint left/arm_2_case_bearing_joint: type fixed, parent left/arm_2_microservo_case, child left/arm_2_case_bearing, origin xyz=0 0 0.072 rpy=0 0 0
- added joint left/base_gripper_joint: type continuous, parent left/core_structure, child left/base_gripper, origin xyz=0 0 0.041 rpy=0 0 ${-pi/2}
- added joint left/core_structure_joint: type fixed, parent left/end_effector_connector, child left/core_structure, origin xyz=0 0 0 rpy=0 0 0
- added joint left/end_effector_connector_joint: type fixed, parent left/arm_2_case_bearing, child left/end_effector_connector, origin xyz=0 0 0 rpy=0 0 0
- added joint left/holdBar_left: type fixed, parent left/base_gripper, child left/holdBar_left, origin xyz=0 -0.02 0.057 rpy=0 0 0
- added joint left/holdBar_right: type fixed, parent left/base_gripper, child left/holdBar_right, origin xyz=0 0.02 0.057 rpy=0 0 0

Commit message: Arm with full gripper

File: arm_description/urdf/4dof.urdf (robot description, URDF)
Before this commit: robot arm4DoF, 17 links, 16 joints
Links:
- added link left/ScrewActuatorGripperCenter; visual mesh filename=package://arm_description/meshes/new_meshes/gripper/ScrewAc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
- added link left/base_gripper_case; visual mesh filename=package://arm_description/meshes/new_meshes/gripper/base_gr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
- added link left/left_bar1; visual mesh filename=package://arm_description/meshes/new_meshes/gripper/bar.stl
- added link left/left_bar2; visual mesh filename=package://arm_description/meshes/new_meshes/gripper/bar.stl
- added link left/left_bar3; visual mesh filename=package://arm_description/meshes/new_meshes/gripper/bar.stl
- added link left/left_bar4; visual mesh filename=package://arm_description/meshes/new_meshes/gripper/bar.stl
- added link left/left_barMini; visual mesh filename=package://arm_description/meshes/new_meshes/gripper/barMini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
- added link left/left_gripper; visual mesh filename=package://arm_description/meshes/new_meshes/gripper/gripper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
- added link left/microservo_FT; visual mesh filename=package://arm_description/meshes/new_meshes/gripper/microse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
- added link left/right_bar1; visual mesh filename=package://arm_description/meshes/new_meshes/gripper/bar.stl
- added link left/right_bar2; visual mesh filename=package://arm_description/meshes/new_meshes/gripper/bar.stl
- added link left/right_bar3; visual mesh filename=package://arm_description/meshes/new_meshes/gripper/bar.stl
- added link left/right_bar4; visual mesh filename=package://arm_description/meshes/new_meshes/gripper/bar.stl
- added link left/right_barMini; visual mesh filename=package://arm_description/meshes/new_meshes/gripper/barMini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
- added link left/right_gripper; visual mesh filename=package://arm_description/meshes/new_meshes/gripper/gripper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
Joints:
- removed joint left/holdBar_left
- removed joint left/holdBar_right
- added joint left/ScrewActuatorGripperCenter_joint: type fixed, parent left/ScrewActuatorGripper, child left/ScrewActuatorGripperCenter, origin xyz=0 0 0 rpy=0 0 0
- added joint left/base_gripper_case_joint: type fixed, parent left/ScrewActuatorGripper, child left/base_gripper_case, origin xyz=0 0 0 rpy=0 0 0
- added joint left/holdBar_left_joint: type fixed, parent left/base_gripper, child left/holdBar_left, origin xyz=0 -0.02 0.057 rpy=0 0 0
- added joint left/holdBar_right_joint: type fixed, parent left/base_gripper, child left/holdBar_right, origin xyz=0 0.02 0.057 rpy=0 0 0
- added joint left/left_bar1_joint: type fixed, parent left/holdBar_left, child left/left_bar1, origin xyz=0.005 -0.012 0.0265 rpy=0 0 0
- added joint left/left_bar2_joint: type fixed, parent left/holdBar_left, child left/left_bar2, origin xyz=0.005 -0.022 0.0265 rpy=0 0 0
- added joint left/left_bar3_joint: type fixed, parent left/holdBar_left, child left/left_bar3, origin xyz=-0.005 -0.012 0.0265 rpy=0 0 0
- added joint left/left_bar4_joint: type fixed, parent left/holdBar_left, child left/left_bar4, origin xyz=-0.005 -0.022 0.0265 rpy=0 0 0
- added joint left/left_barMini_joint: type fixed, parent left/left_bar1, child left/left_barMini, origin xyz=-0.0043 0 0.0155 rpy=0 0 0
- added joint left/left_gripper_joint: type continuous, parent left/left_barMini, child left/left_gripper, origin xyz=0 0 0.025 rpy=0 0 0
- added joint left/microservo_FT_joint: type fixed, parent left/base_gripper, child left/microservo_FT, origin xyz=0 0 0.057 rpy=${pi/2} 0 ${pi/2}
- added joint left/right_bar1_joint: type fixed, parent left/holdBar_right, child left/right_bar1, origin xyz=0.005 0.012 0.0265 rpy=0 0 0
- added joint left/right_bar2_joint: type fixed, parent left/holdBar_right, child left/right_bar2, origin xyz=0.005 0.022 0.0265 rpy=0 0 0
- added joint left/right_bar3_joint: type fixed, parent left/holdBar_right, child left/right_bar3, origin xyz=-0.005 0.012 0.0265 rpy=0 0 0
- added joint left/right_bar4_joint: type fixed, parent left/holdBar_right, child left/right_bar4, origin xyz=-0.005 0.022 0.0265 rpy=0 0 0
- added joint left/right_barMini_joint: type fixed, parent left/right_bar1, child left/right_barMini, origin xyz=-0.0043 0 0.0155 rpy=0 0 0
- added joint left/right_gripper_joint: type continuous, parent left/right_barMini, child left/right_gripper, origin xyz=0 0 0.025 rpy=0 0 ${pi}
- joint left/ScrewActuatorGripper_joint: origin xyz=0 0 0.055 rpy=0 0 0 -> xyz=0 0 0 rpy=${-pi/2} 0 0; parent left/base_gripper -> left/microservo_FT

Commit message: Detector

File: arm_description/urdf/4dof.urdf (robot description, URDF)
Before this commit: robot arm4DoF, 32 links, 31 joints
Links:
- added link right/ScrewActuatorGripper; visual mesh filename=package://arm_description/meshes/new_meshes/gripper/ScrewAc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
- added link right/ScrewActuatorGripperCenter; visual mesh filename=package://arm_description/meshes/new_meshes/gripper/ScrewAc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
- added link right/arm_0_attachment; visual mesh filename=package://arm_description/meshes/new_meshes/arm_0_attachmen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
- added link right/arm_0_bottom; visual mesh filename=package://arm_description/meshes/new_meshes/arm_0_bottom.stl
- added link right/arm_0_bottom_case; visual mesh filename=package://arm_description/meshes/new_meshes/arm_0_bottom_ca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
- added link right/arm_0_bottom_top_lock; visual mesh filename=package://arm_description/meshes/new_meshes/arm_0_bottom_to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
- added link right/arm_0_top; visual mesh filename=package://arm_description/meshes/new_meshes/arm_0_top.stl
- added link right/arm_1; visual mesh filename=package://arm_description/meshes/new_meshes/arm_1.stl
- added link right/arm_1_case; visual mesh filename=package://arm_description/meshes/new_meshes/arm_1_case.stl
- added link right/arm_2_case_bearing; visual mesh filename=package://arm_description/meshes/new_meshes/arm_2_case_bear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
- added link right/arm_2_microservo; visual mesh filename=package://arm_description/meshes/new_meshes/arm_2_microserv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
- added link right/arm_2_microservo_case; visual mesh filename=package://arm_description/meshes/new_meshes/arm_2_microserv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
- added link right/base_gripper; visual mesh filename=package://arm_description/meshes/new_meshes/gripper/base_gr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
- added link right/base_gripper_case; visual mesh filename=package://arm_description/meshes/new_meshes/gripper/base_gr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
- added link right/core_structure; visual mesh filename=package://arm_description/meshes/new_meshes/gripper/core_st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
- added link right/end_effector_connector; visual mesh filename=package://arm_description/meshes/new_meshes/end_effector_co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
- added link right/holdBar_left; visual mesh filename=package://arm_description/meshes/new_meshes/gripper/holdBar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
- added link right/holdBar_right; visual mesh filename=package://arm_description/meshes/new_meshes/gripper/holdBar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
- added link right/left_bar1; visual mesh filename=package://arm_description/meshes/new_meshes/gripper/bar.stl
- added link right/left_bar2; visual mesh filename=package://arm_description/meshes/new_meshes/gripper/bar.stl
- added link right/left_bar3; visual mesh filename=package://arm_description/meshes/new_meshes/gripper/bar.stl
- added link right/left_bar4; visual mesh filename=package://arm_description/meshes/new_meshes/gripper/bar.stl
- added link right/left_barMini; visual mesh filename=package://arm_description/meshes/new_meshes/gripper/barMini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
- added link right/left_gripper; visual mesh filename=package://arm_description/meshes/new_meshes/gripper/gripper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
- added link right/microservo_FT; visual mesh filename=package://arm_description/meshes/new_meshes/gripper/microse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
- added link right/right_bar1; visual mesh filename=package://arm_description/meshes/new_meshes/gripper/bar.stl
- added link right/right_bar2; visual mesh filename=package://arm_description/meshes/new_meshes/gripper/bar.stl
- added link right/right_bar3; visual mesh filename=package://arm_description/meshes/new_meshes/gripper/bar.stl
- added link right/right_bar4; visual mesh filename=package://arm_description/meshes/new_meshes/gripper/bar.stl
- added link right/right_barMini; visual mesh filename=package://arm_description/meshes/new_meshes/gripper/barMini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
- added link right/right_gripper; visual mesh filename=package://arm_description/meshes/new_meshes/gripper/gripper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
Joints:
- added joint right/ScrewActuatorGripperCenter_joint: type fixed, parent right/ScrewActuatorGripper, child right/ScrewActuatorGripperCenter, origin xyz=0 0 0 rpy=0 0 0
- added joint right/ScrewActuatorGripper_joint: type fixed, parent right/microservo_FT, child right/ScrewActuatorGripper, origin xyz=0 0 0 rpy=${-pi/2} 0 0
- added joint right/arm_0_attachment_joint: type fixed, parent base_link, child right/arm_0_attachment, origin xyz=0 -0.2 0 rpy=0 0 0
- added joint right/arm_0_bottom_case_joint: type fixed, parent right/arm_0_bottom, child right/arm_0_bottom_case, origin xyz=-0.017 0 0 rpy=0 0 0
- added joint right/arm_0_bottom_joint: type continuous, parent right/arm_0_bottom_top_lock, child right/arm_0_bottom, origin xyz=0 0 -0.005 rpy=0 ${-pi/2} ${-pi/2}
- added joint right/arm_0_bottom_top_lock_joint: type fixed, parent right/arm_0_top, child right/arm_0_bottom_top_lock, origin xyz=0 0 0 rpy=0 0 0
- added joint right/arm_0_top_joint: type fixed, parent right/arm_0_attachment, child right/arm_0_top, origin xyz=0 0 -0.03 rpy=0 0 0
- added joint right/arm_1_case_joint: type fixed, parent right/arm_1, child right/arm_1_case, origin xyz=0 0 0.145 rpy=0 0 0
- added joint right/arm_1_joint: type continuous, parent right/arm_0_bottom_case, child right/arm_1, origin xyz=0 0 0 rpy=0 ${3*pi/2} 0
- added joint right/arm_2_case_bearing_joint: type fixed, parent right/arm_2_microservo_case, child right/arm_2_case_bearing, origin xyz=0 0 0.072 rpy=0 0 0
- added joint right/arm_2_microservo_case_joint: type fixed, parent right/arm_2_microservo, child right/arm_2_microservo_case, origin xyz=0 0 0.057 rpy=0 0 0
- added joint right/arm_2_microservo_joint: type continuous, parent right/arm_1_case, child right/arm_2_microservo, origin xyz=0 0 0.0085 rpy=0 0 0
- added joint right/base_gripper_case_joint: type fixed, parent right/ScrewActuatorGripper, child right/base_gripper_case, origin xyz=0 0 0 rpy=0 0 0
- added joint right/base_gripper_joint: type continuous, parent right/core_structure, child right/base_gripper, origin xyz=0 0 0.041 rpy=0 0 ${-pi/2}
- added joint right/core_structure_joint: type fixed, parent right/end_effector_connector, child right/core_structure, origin xyz=0 0 0 rpy=0 0 0
- added joint right/end_effector_connector_joint: type fixed, parent right/arm_2_case_bearing, child right/end_effector_connector, origin xyz=0 0 0 rpy=0 0 0
- added joint right/holdBar_left_joint: type fixed, parent right/base_gripper, child right/holdBar_left, origin xyz=0 -0.02 0.057 rpy=0 0 0
- added joint right/holdBar_right_joint: type fixed, parent right/base_gripper, child right/holdBar_right, origin xyz=0 0.02 0.057 rpy=0 0 0
- added joint right/left_bar1_joint: type fixed, parent right/holdBar_left, child right/left_bar1, origin xyz=0.005 -0.012 0.0265 rpy=0 0 0
- added joint right/left_bar2_joint: type fixed, parent right/holdBar_left, child right/left_bar2, origin xyz=0.005 -0.022 0.0265 rpy=0 0 0
- added joint right/left_bar3_joint: type fixed, parent right/holdBar_left, child right/left_bar3, origin xyz=-0.005 -0.012 0.0265 rpy=0 0 0
- added joint right/left_bar4_joint: type fixed, parent right/holdBar_left, child right/left_bar4, origin xyz=-0.005 -0.022 0.0265 rpy=0 0 0
- added joint right/left_barMini_joint: type fixed, parent right/left_bar1, child right/left_barMini, origin xyz=-0.0043 0 0.0155 rpy=0 0 0
- added joint right/left_gripper_joint: type continuous, parent right/left_barMini, child right/left_gripper, origin xyz=0 0 0.025 rpy=0 0 0
- added joint right/microservo_FT_joint: type fixed, parent right/base_gripper, child right/microservo_FT, origin xyz=0 0 0.057 rpy=${pi/2} 0 ${pi/2}
- added joint right/right_bar1_joint: type fixed, parent right/holdBar_right, child right/right_bar1, origin xyz=0.005 0.012 0.0265 rpy=0 0 0
- added joint right/right_bar2_joint: type fixed, parent right/holdBar_right, child right/right_bar2, origin xyz=0.005 0.022 0.0265 rpy=0 0 0
- added joint right/right_bar3_joint: type fixed, parent right/holdBar_right, child right/right_bar3, origin xyz=-0.005 0.012 0.0265 rpy=0 0 0
- added joint right/right_bar4_joint: type fixed, parent right/holdBar_right, child right/right_bar4, origin xyz=-0.005 0.022 0.0265 rpy=0 0 0
- added joint right/right_barMini_joint: type fixed, parent right/right_bar1, child right/right_barMini, origin xyz=-0.0043 0 0.0155 rpy=0 0 0
- added joint right/right_gripper_joint: type continuous, parent right/right_barMini, child right/right_gripper, origin xyz=0 0 0.025 rpy=0 0 ${pi}
