Commit message: uav_hecatonquiros

File: arm_description/urdf/one_arm.urdf (robot description, URDF)
Before this commit: robot arm4DoF, 6 links, 5 joints
Links:
- link arm_0_bottom: geometry visual mesh filename=package://arm_description/meshes/old_meshes/arm_0_bottom.stl scale=0.01 0.01 0.01
- link arm_0_closing_case: geometry visual mesh filename=package://arm_description/meshes/old_meshes/arm_0_closing_c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 scale=0.01 0.01 0.01
- link arm_0_top: geometry collision box size=1 1 0.67; visual mesh filename=package://arm_description/meshes/old_meshes/arm_0_top.stl scale=0.01 0.01 0.01
- link arm_1: geometry collision box size=0.73 0.3 1.0; visual mesh filename=package://arm_description/meshes/old_meshes/arm_1.stl scale=0.01 0.01 0.01
- link arm_2: geometry collision box size=0.86 0.3 1.2; visual mesh filename=package://arm_description/meshes/old_meshes/arm_2.stl scale=0.01 0.01 0.01
